File: keyboard.sch (KiCad schematic (older format))
At the start: 84 parts, among them IC1 ATMEGA32U4, J1 MINI, P1 CONN_1, P10 CONN_1, P11 CONN_1, P12 CONN_1, P13 CONN_1, P14 CONN_1, P15 CONN_1, P16 CONN_1, P17 CONN_1, P18 CONN_1, P19 CONN_1, P2 CONN_1, P20 CONN_1, P21 CONN_1, P22 CONN_1, P23 CONN_1, P24 CONN_1, P25 CONN_1, P26 CONN_1, P27 CONN_1, P28 CONN_1, P29 CONN_1, P3 CONN_1, P30 CONN_1, P31 CONN_1, P32 CONN_1, P33 CONN_1, P34 CONN_1, P35 CONN_1, P36 CONN_1, P37 CONN_1, P38 CONN_1, P39 CONN_1, P4 CONN_1, P40 CONN_1, P41 CONN_1, P42 CONN_1, P5 CONN_1, P6 CONN_1, P7 CONN_1, P8 CONN_1, P9 CONN_1, X1 ASX3F

Commit message: 修改usb接口为type c
Parts:
- removed J1: MINI, usb:67503, symbol USBMINI_B05
- renumbered C8 to C1, C4 to C2, C5 to C3, C1 to C4, C6 to C5, C7 to C6, C3 to C7, C2 to C8, DF3 to DF1, DF20 to DF10, DF10 to DF11, DF11 to DF12, DF232 to DF2, DF231 to DF3, DF23 to DF4, DF221 to DF5, DF22 to DF6, DF211 to DF7, DF21 to DF8, DF201 to DF9, P21 to P10, P22 to P11, P11 to P12, P12 to P13, P13 to P14, P14 to P15, P15 to P16, P23 to P17, P24 to P18, P25 to P19, P3 to P2, P26 to P20, P27 to P21, P28 to P22, P29 to P23, P30 to P24, P31 to P25, P32 to P26, P33 to P27, P34 to P28, P35 to P29, P5 to P3, P36 to P30, P37 to P31, P38 to P32, P39 to P33, P40 to P34, P41 to P35, P42 to P36, P7 to P37, P8 to P38, P9 to P39, P2 to P4, P10 to P40, P16 to P41, P17 to P42, P4 to P5, P18 to P7, P19 to P8, P20 to P9, R6 to R10, R7 to R11, R8 to R12, R9 to R13, R12 to R14, R5 to R3, R3 to R4, R15 to R5, R14 to R6, R13 to R7, R11 to R8, R10 to R9
Connections:
- wire segments 205 -> 203
- no-connect marks 5 -> 4

Commit message: 增加一列F功能区 增加TrackPiont模块,同时增加ffc排线接口 右移右侧键布局
Parts:
- removed DF1, DF10, DF11, DF12, DF9, DW1, DW2, DW3, DW4: LED, mx1a:MX1A-led_no3d, symbol LED
- removed DF2, DF3, DF4, DF5, DF6, DF7, DF8: LED, symbol LED
- removed P12, P13, P14, P15, P16, P39, P40, P41, P42: CONN_1, symbol CONN_1
- removed R10, R11, R12, R13, R14, R5, R6, R7, R8, R9: R, symbol R
- added C_TP1: 2.2uf, Capacitors_SMD:C_1206, symbol CP1
- added R_TP1, R_TP2: 4.7k, 0805:0805R, symbol R
- added R_TP3: 100k, 0805:0805R, symbol R
- added TP_J1: CONN_8, connectors:connector-ffc-8p, symbol CONN_8
- added TP_J2: CONN_4, connectors:connector-ffc-4p, symbol CONN_4
- renumbered C4 to C1, C8 to C2, C7 to C3, C2 to C4, C3 to C5, C5 to C6, C6 to C7, C1 to C8, P35 to P10, P31 to P11, P36 to P12, P7 to P18, P8 to P19, P4 to P2, P9 to P20, P10 to P21, P11 to P22, P17 to P23, P18 to P24, P19 to P25, P20 to P26, P21 to P27, P22 to P28, P23 to P29, P2 to P3, P24 to P30, P25 to P31, P26 to P32, P27 to P33, P28 to P34, P29 to P35, P30 to P36, P5 to P4, P3 to P5, P32 to P7, P33 to P8, P34 to P9, R4 to R3, R3 to R4
Connections:
- net labels added: btn1, btn2, btn3, clk, data, row6, rst, tp_clk, tp_data, vcc
- net labels removed: GPIO0, GPIO1, GPIO2, GPIO3
- wire segments 203 -> 161
- no-connect marks 4 -> 5
Other:
- note added: "jtag connector (bottom)"
- note removed: "Backlight expansion\nconnector (top)"
- note removed: "Universal expansion\nconnector (bottom)"

Commit message: 第一版 修改了鼠标三键错位 TrackPiont模块ffc接口位置修改方便连接
Parts:
- removed P1, P10, P11, P12, P18, P19, P2, P20, P21, P22, P23, P24, P25, P26, P27, P28, P29, P3, P30, P31, P32, P33, P34, P35, P36, P37, P38, P4, P5, P6, P7, P8, P9: CONN_1, symbol CONN_1
- added P1: CONN_3X2, Connectors_IDC:IDC-Header_2x03_Pitch2.54mm_Straight, symbol CONN_3X2
- added P2: DIL24, connectors:ffc-0.5mm-24p, symbol DIL24
Connections:
- net labels added: lcol1, lcol10, lcol11, lcol12, lcol13, lcol14, lcol2, lcol3, lcol4, lcol5, lcol6, lcol7, lcol8, lcol9, lrow1, lrow2, lrow3, lrow4, lrow5, lrow6
- wire segments 161 -> 177

Commit message: 一些改动
Parts:
- removed P2: DIL24, connectors:ffc-0.5mm-24p, symbol DIL24
